Commit message: Make the simulation physically real, and drive the base
The sim previously spawned a robot that could not hold still or move
correctly. Four separate causes, each found by measurement:

The arm sagged into the sensor gantry. xarm6_traj_controller claims both
position and velocity command interfaces, and gz_ros2_control picks one
control law per joint by fixed priority, so velocity always won. A
finished trajectory holds velocity 0 with no feedback term, which is an
open loop against gravity: joint2/3 sagged a little further every cycle
until the arm folded into the pedestal. Claiming position only lets its
proportional loop see the error. The stock gain is left alone
deliberately; update_rate is already baked into the product, and raising
it just makes the joints hunt.

The whole platform was massless. Nothing in the description carried an
<inertial>, so gz substituted a ~1 kg placeholder and an 18 kg arm could
shove the base around. Chassis and gantry now carry mass and inertia,
with the gantry centre of mass low and aft where the battery is.

Nothing drove the base, and base_link is the URDF root with no joint
above it, so it was a free-floating body held up by ground contact
alone. Without wheels it is now welded to a world link; with them it
rides on four steered wheels. The two are opposites, not companions.

Wheel geometry is measured off ranger_mini_v3_cad.stl by circle fit to
the lower arc of each tyre, not taken from a datasheet: radius 0.1026,
wheelbase 0.494, track 0.3704, all within 2 mm and agreeing with the
published figures. The tread lands on ground_z_nom to seven decimals.
ranger_envelope had to be cut back to the chassis proper, because as a
whole-vehicle bound its underside sat 5.5 cm BELOW the tread and the
chassis grounded out with the wheels spinning in the air.

Four-wheel independent steering needs no mode switch. Pointing each
wheel along v + w x r and spinning it at that magnitude gives crab, spin
and Ackermann from one formula; ros2_control's steering library cannot
express it because every controller there assumes a fixed rear axle.

dartsim, not bullet-featherstone. bullet implements a joint velocity
command as a rigid motor constraint that never disengages
(gazebosim/gz-sim#2729), so four wheels and four steer joints
over-determine the chassis and it refuses to yaw: a commanded 229 deg
spin gave 0.5 deg, and friction was irrelevant because a wheel that
cannot slip does not care. The same model on dartsim spins in place.

Measured, drive_base:=true: forward 91%, crab 90%, spin 204 of 229 deg
with zero translation, arcs correct. Arm tracks to ~1e-6 rad and the
base moves 0.19 mm during a full arm sweep.

NOTE: the gripper needs a matching change to xarm_gripper.ros2_control
.xacro, declaring the five follower joints with mimic="true" so
ros2_control drives them instead of relying on engine mimic support,
which dartsim lacks (gz-physics#432). That file lives under
src/xarm_ros2/, which this repo gitignores, so it is NOT in this commit
and a fresh vcs import will not have it. See docs/TODO.md.

File: src/ranger_xarm_description/urdf/ranger_xarm.urdf.xacro (robot description, xacro)
@@ -5,4 +5,5 @@
   <xacro:include filename="$(find ranger_xarm_description)/urdf/sensor_frames.xacro"/>
   <xacro:include filename="$(find ranger_xarm_description)/urdf/laptop_collision.xacro"/>
+  <xacro:include filename="$(find ranger_xarm_description)/urdf/ranger_wheels.xacro"/>
   <xacro:arg name="use_xarm" default="true"/>
   <xacro:arg name="use_static_geometry" default="true"/>
@@ -33,4 +34,21 @@
   <xacro:arg name="os0_dx" default="0.0"/><xacro:arg name="os0_dy" default="0.0"/><xacro:arg name="os0_dz" default="0.0"/>
   <xacro:arg name="d435_dx" default="0.0"/><xacro:arg name="d435_dy" default="0.0"/><xacro:arg name="d435_dz" default="0.0"/>
+  <!-- Base drive. Following the same rule the arm already uses; simulation
+       changes xacro arguments, not the model; both default to the
+       hardware/planning behaviour, and only the gz launch turns them over:
+         use_wheels         adds the 4WIS steer+roll joints and their
+                            ros2_control interfaces. Off by default because
+                            no hardware driver here publishes those joint
+                            states, and an unpublished joint is a frame that
+                            silently sits at zero in RViz and MoveIt.
+         fix_base_to_world  welds base_link down. On by default, because
+                            without wheels base_link is a free-floating root
+                            link held up by nothing but ground contact, and
+                            the arm's reaction forces walk it across the
+                            floor. Turn it OFF whenever use_wheels is on;
+                            they are opposites, not companions. -->
+  <xacro:arg name="use_wheels" default="false"/>
+  <xacro:arg name="fix_base_to_world" default="true"/>
+  <xacro:arg name="wheels_ros2_control_plugin" default="gz_ros2_control/GazeboSimSystem"/>
   <xacro:arg name="use_laptop_collision" default="true"/>
   <xacro:arg name="laptop_width" default="0.36"/><xacro:arg name="laptop_depth" default="0.25"/>
@@ -39,4 +57,23 @@
   <xacro:arg name="laptop_clearance" default="0.015"/>
   <link name="base_link"/>
+  <!-- base_link is the URDF root with no joint above it, so gz-sim spawns it
+       as a free-floating 6-DOF body held up by nothing but ground contact.
+       With no wheels to carry it, the arm's reaction forces couple into that
+       floating body every step and walk it across the floor. Welding it to a
+       "world" link; the convention gz-sim's URDF to SDF conversion
+       recognises for a stationary base; makes it a fixed pedestal, which
+       is what MoveIt planning and display.launch.py already assume. -->
+  <xacro:if value="$(arg fix_base_to_world)">
+    <link name="world"/>
+    <joint name="world_to_base_link" type="fixed">
+      <parent link="world"/>
+      <child link="base_link"/>
+    </joint>
+  </xacro:if>
+  <xacro:if value="$(arg use_wheels)">
+    <xacro:ranger_wheels parent="base_link" ground_z="${ground_z_nom}"/>
+    <xacro:ranger_wheels_ros2_control name="ranger_base"
+      plugin="$(arg wheels_ros2_control_plugin)"/>
+  </xacro:if>
   <!-- Ground-projection reference. Kept as a child of base_link so the
        Ranger odometry publisher can later own odom -> base_link without a
@@ -49,5 +86,6 @@
   </joint> -->
   <xacro:if value="$(arg use_static_geometry)">
-    <xacro:ranger_static_geometry parent="base_link" use_collision="$(arg use_static_collision)"/>
+    <xacro:ranger_static_geometry parent="base_link" use_collision="$(arg use_static_collision)"
+      wheels_modelled="$(arg use_wheels)"/>
   </xacro:if>
   <link name="xarm_mount_link"/>

File: src/ranger_xarm_description/urdf/static_geometry.xacro (robot description, xacro)
@@ -1,6 +1,20 @@
 <?xml version="1.0"?>
 <robot xmlns:xacro="http://www.ros.org/wiki/xacro">
-  <xacro:macro name="ranger_static_geometry" params="parent:='base_link' use_collision:=true">
+  <xacro:macro name="ranger_static_geometry" params="parent:='base_link' use_collision:=true wheels_modelled:=false">
     <link name="ranger_cad_link">
+      <!-- Chassis mass. Nothing in this description carried an <inertial> at
+           all, which means the whole platform was massless in physics: gz
+           falls back to a ~1 kg placeholder, so an 18 kg arm swinging on top
+           could shove the base around, and a massless wheel has no normal
+           force and therefore no traction. AgileX publish 63 kg for a loaded
+           Ranger Mini; 47 kg here leaves room for the 4x3 kg wheels and
+           4x1 kg steering knuckles in ranger_wheels.xacro. Inertia is the
+           solid-box equivalent of the ranger_envelope collision, taken about
+           the same centre. -->
+      <inertial>
+        <origin xyz="-0.001 0 -0.181436" rpy="0 0 0"/>
+        <mass value="47.0"/>
+        <inertia ixx="1.6086" ixy="0" ixz="0" iyy="3.1592" iyz="0" izz="3.5065"/>
+      </inertial>
       <visual name="ranger_cad_visual">
         <geometry>
@@ -10,8 +24,26 @@
       </visual>
       <xacro:if value="${use_collision}">
-        <collision name="ranger_envelope">
-          <origin xyz="-0.001000 0 -0.181436" rpy="0 0 0"/>
-          <geometry><box size="0.803706 0.500020 0.400891"/></geometry>
-        </collision>
+        <!-- ranger_envelope is the whole-vehicle bounding box, wheels
+             included, so its underside sits at base_link z=-0.3819: 5.5 cm
+             BELOW the wheel tread at -0.3270. With no wheel collisions that
+             is merely conservative, and the platform rests on the box.
+             Once ranger_wheels.xacro provides real tyre collisions it is
+             actively wrong; the box grounds out first and holds the wheels
+             in the air, where they spin freely and the robot cannot drive.
+             So when wheels are modelled the envelope is cut back to the
+             chassis proper, whose underside measures -0.2514 in the CAD
+             mesh (76 mm ground clearance, matching the published spec). -->
+        <xacro:if value="${wheels_modelled}">
+          <collision name="ranger_envelope">
+            <origin xyz="-0.001000 0 -0.116180" rpy="0 0 0"/>
+            <geometry><box size="0.803706 0.500020 0.270360"/></geometry>
+          </collision>
+        </xacro:if>
+        <xacro:unless value="${wheels_modelled}">
+          <collision name="ranger_envelope">
+            <origin xyz="-0.001000 0 -0.181436" rpy="0 0 0"/>
+            <geometry><box size="0.803706 0.500020 0.400891"/></geometry>
+          </collision>
+        </xacro:unless>
       </xacro:if>
     </link>
@@ -21,4 +53,15 @@
     </joint>
     <link name="custom_structure_link">
+      <!-- Gantry, arm pedestal, EcoFlow pack, laptop stand and control box.
+           Estimated, not weighed: the battery dominates at roughly half of
+           it. The centre of mass sits low and aft, where the pack and power
+           mount are, NOT at the gantry mid-height; putting it at the
+           geometric centre of the gantry would invent a tippy robot that
+           the real platform is not. -->
+      <inertial>
+        <origin xyz="-0.150 0 0.350" rpy="0 0 0"/>
+        <mass value="25.0"/>
+        <inertia ixx="3.134" ixy="0" ixz="0" iyy="3.817" iyz="0" izz="1.724"/>
+      </inertial>
       <visual name="custom_structure_visual">
         <geometry>

Commit message: Enable base_footprint and give the EKF its TF edge
base_footprint was commented out of the description while
ranger_xarm_bringup's EKF is configured with base_link_frame:
base_footprint and publish_tf: true. The EKF was therefore publishing
into a frame that did not exist in simulation. It is now a real link:
massless and geometry-free, so sdformat merges it into base_link during
conversion and it costs gz nothing, while robot_state_publisher still
puts the frame on TF because it reads the URDF rather than the SDF.

wheel_odometry.py now names base_footprint as its child frame to match,
and sim.launch.py gains odom_tf, default true, to be set false whenever
the EKF runs. Two publishers on one TF edge is not reported as an error;
TF just returns whichever arrived last, which is the kind of thing that
is discovered much later and blamed on something else.

With that in place the EKF could be run against the simulator for the
first time, and it does not track heading. On empty_ground over a drive
with 138.0 deg of real rotation:

  wheel odometry    0.007 m   0.11% of path    +0.17 deg
  EKF (odom+gyro)   5.799 m  86.76% of path  -138.00 deg

The EKF's orientation stays exactly identity and its yaw rate stays
exactly zero. -138.00 against +138.0 is not drift, it is the filter never
rotating. Wheel odometry on the same run is 0.11%, so /odom is sound.

This is NOT a verdict on the EKF and is not being presented as one. It
has never been run against this simulator before today, so a wiring
fault on the simulation side is at least as likely as a filter fault, and
the hardware behaviour is untouched by any of this. What is recorded in
docs/TODO.md is the evidence and the ruling-out: TF resolves, the frame
id matches, the vyaw covariance is 1e-05 rather than -1, sim time is
consistent across clock, IMU, corrector and odom, the config indices are
the intended wheels-for-speed gyro-for-turning split, and the raw gyro
reads 1.36 rad/s during a commanded spin. Why a valid measurement
produces no yaw is still open.

One thing found along the way IS a defect. imu_yaw_bias_corrector seeds a
gyro-z bias of +0.3350 deg/s measured on hardware, and max_bias_step is
0.0035 rad/s (0.2005 deg/s). Against an IMU whose true bias is zero, the
correction needed is larger than the step it will accept, so it rejects
every re-estimate and stays permanently wrong:

  seeded gyro-z bias +0.3350 deg/s
  rejecting gyro bias jump of -0.3350 deg/s (limit 0.2005)

The guard that protects it from a bad stationary sample locks it onto the
seed against any IMU whose bias differs by more than 0.2 deg/s. That is
worth fixing on its own account.

None of this was visible while /odom was ground truth.

File: src/ranger_xarm_description/urdf/ranger_xarm.urdf.xacro (robot description, xacro)
@@ -82,13 +82,20 @@
       plugin="$(arg wheels_ros2_control_plugin)"/>
   </xacro:if>
-  <!-- Ground-projection reference. Kept as a child of base_link so the
-       Ranger odometry publisher can later own odom -> base_link without a
-       competing TF parent. -->
-  <!-- <link name="base_footprint"/>
+  <!-- Ground-projection reference, and the frame the state estimator
+       localises. ranger_xarm_bringup's EKF is configured with
+       base_link_frame: base_footprint and publish_tf: true, so it owns
+       odom -> base_footprint; nothing else may publish that edge. This
+       link is the other end of it, and while it was commented out the
+       EKF was publishing into a frame that did not exist in simulation.
+       Massless and geometry-free on purpose. sdformat merges a fixed
+       child like this into base_link during conversion, so it costs gz
+       nothing, and the frame still reaches TF because
+       robot_state_publisher reads the URDF rather than the SDF. -->
+  <link name="base_footprint"/>
   <joint name="base_to_base_footprint" type="fixed">
     <parent link="base_link"/>
     <child link="base_footprint"/>
     <origin xyz="0 0 ${ground_z_nom}" rpy="0 0 0"/>
-  </joint> -->
+  </joint>
   <xacro:if value="$(arg use_static_geometry)">
     <xacro:ranger_static_geometry parent="base_link" use_collision="$(arg use_static_collision)"

Commit message: Make base_footprint the tree root, fixing the EKF heading fault
base_footprint was enabled as a child of base_link while the EKF is
configured with base_link_frame: base_footprint and publish_tf: true, so
it publishes odom -> base_footprint. The frame had two parents. tf2
allows exactly one, so the estimator's edge orphaned
robot_state_publisher's, and every lookup that had to cross the break
failed.

The IMU is in os_imu, under base_link, on the far side of that break, so
every IMU measurement was discarded. odom0 was unaffected because its
child_frame_id is already base_footprint and needs no lookup. The filter
therefore fused wheel velocity perfectly and never rotated.

  wheel odometry    0.007 m   0.11% of path    +0.17 deg
  EKF  (before)     6.219 m  91.97% of path  -147.39 deg
  EKF  (after)      0.093 m   1.39% of path    -0.01 deg

base_footprint is now the root with base_link as its child, which is the
conventional layout for a mobile base and the one the EKF config already
assumed. The world weld moves to the root for the same reason: welding
base_link would have given it two parents and broken the tree the same
way.

The original comment on this block was right and I should have read it as
a constraint rather than a note. It said base_footprint was kept as a
child of base_link "so the Ranger odometry publisher can later own
odom -> base_link without a competing TF parent". Enabling it in that
orientation created exactly the competing parent it warned about.

Three things made this expensive to find, all recorded in docs/TODO.md.
Nothing reports it: the filter runs, publishes at its configured rate and
its diagnostics report it healthy, with the discard visible only under
debug as "Could not transform measurement into base_footprint". The
transform resolves perfectly from any other process, because the second
parent exists only while the estimator is publishing, so every external
check said TF was fine. And half the inputs keep working, so the output
looks plausible rather than absent.

The discriminator that found it: point base_link_frame at the frame the
sensor already hangs off. If the measurement starts being fused, the
target frame is the problem rather than the sensor, the data or the
filter.

File: src/ranger_xarm_description/urdf/ranger_xarm.urdf.xacro (robot description, xacro)
@@ -74,5 +74,8 @@
     <joint name="world_to_base_link" type="fixed">
       <parent link="world"/>
-      <child link="base_link"/>
+      <!-- base_footprint is the root now, so the weld goes there. Welding
+           base_link instead would give it two parents and break the tree
+           the same way base_footprint used to be broken. -->
+      <child link="base_footprint"/>
     </joint>
   </xacro:if>
@@ -82,19 +85,29 @@
       plugin="$(arg wheels_ros2_control_plugin)"/>
   </xacro:if>
-  <!-- Ground-projection reference, and the frame the state estimator
-       localises. ranger_xarm_bringup's EKF is configured with
-       base_link_frame: base_footprint and publish_tf: true, so it owns
-       odom -> base_footprint; nothing else may publish that edge. This
-       link is the other end of it, and while it was commented out the
-       EKF was publishing into a frame that did not exist in simulation.
-       Massless and geometry-free on purpose. sdformat merges a fixed
-       child like this into base_link during conversion, so it costs gz
-       nothing, and the frame still reaches TF because
-       robot_state_publisher reads the URDF rather than the SDF. -->
+  <!-- Ground-projection reference, and the ROOT of the robot.
+       base_footprint is the parent of base_link, not its child. That
+       ordering is not cosmetic, it is what keeps the TF tree legal.
+       ranger_xarm_bringup's EKF is configured with base_link_frame:
+       base_footprint and publish_tf: true, so it publishes
+       odom -> base_footprint. If base_footprint were also a child of
+       base_link, as it was when this block was first written, the frame
+       would have two parents: one from the estimator and one from
+       robot_state_publisher. tf2 requires exactly one. The second edge
+       orphans the first, and every lookup that has to cross it fails.
+       That failure is close to invisible. The estimator still runs, still
+       publishes, and reports itself healthy; it simply discards every
+       measurement whose frame sits on the wrong side of the break. Here
+       that was the IMU, in os_imu under base_link, so the filter fused
+       wheel velocity happily and never rotated: 138 degrees of real
+       heading change came out as zero, with no warning anywhere outside
+       robot_localization's debug log.
+       With base_footprint as the root, the estimator owns
+       odom -> base_footprint, this joint owns base_footprint ->
+       base_link, and nothing is shared. -->
   <link name="base_footprint"/>
-  <joint name="base_to_base_footprint" type="fixed">
-    <parent link="base_link"/>
-    <child link="base_footprint"/>
-    <origin xyz="0 0 ${ground_z_nom}" rpy="0 0 0"/>
+  <joint name="base_footprint_to_base_link" type="fixed">
+    <parent link="base_footprint"/>
+    <child link="base_link"/>
+    <origin xyz="0 0 ${-ground_z_nom}" rpy="0 0 0"/>
   </joint>
   <xacro:if value="$(arg use_static_geometry)">
