Commit message: Make the wheels visible, and fix the wheel radius
The wheels never moved on screen. ranger_mini_v3_cad.stl is the whole
vehicle as one mesh with its wheels moulded in, and it hangs off
base_link, so the wheels you could see were welded to the chassis; the
wheel links that actually roll and steer carried no <visual> at all,
only a collision sphere and an inertial. The platform drove correctly
and looked completely static.

That was a deliberate trade recorded in ranger_wheels.xacro ("a second
set of visuals would render eight ... verify steering from joint states,
not the GUI"). It is the wrong trade for a simulator you are meant to
watch, and it does not have to be made: scripts/split_wheel_meshes.py
cuts the four wheels out of the CAD as their own meshes and leaves a
body mesh behind, so each wheel goes to the link it belongs to and there
are still only four. static_geometry.xacro draws the body mesh when
wheels_modelled, the original otherwise, so the wheel-less build is
unchanged.

The wheels are separate connected components in the STL, as CAD assembly
exports usually are, so the split is exact rather than a distance
threshold cutting through the suspension: 9040+9036+9032+9040 wheel
triangles and 156590 body, summing to the original 192738. Each wheel is
re-origined on an axis fitted from its own tread so it spins true
instead of wobbling.

A cylinder primitive would not have fixed this. A featureless cylinder
rotating about its own axis is indistinguishable from a stationary one;
it is the spokes and tread that make the rotation legible.

Isolating the tyre also showed the radius was wrong. It reads as a clean
cylinder of 100.036 mm (99.9th percentile 100.032), and the lowest point
of the whole CAD is -327.029 mm, exactly ground_z. Those give an axle at
-226.993 mm, which is where fitting the rear tyre's axis independently
puts it, -226.998. The description said 0.1026 m, from an earlier circle
fit to "the lower arc of each tyre" that had picked up the suspension
sitting inside the same envelope.

AgileX's own assets corroborate it independently: wheel_v3.dae in
agilexrobotics/ugv_gazebo_sim (ranger_mini_v3) is a unit-sphere-scaled
mesh whose node matrix is 0.1003675, i.e. a 100.37 mm wheel, and 200 mm
is the platform's stock size. Note their ranger_mini.xacro separately
declares wheel_radius 0.09, which is 10% under their own visual mesh, so
that number is not the one to copy.

2.6 mm is invisible on screen but it scales every wheel speed the
kinematics computes, so on hardware the platform would have run 2.6%
fast. wheel_radius and ranger_4wis_controller's default both corrected.
Nothing changes in sim, because the collision sphere and the controller
move together.

Verified in Gazebo with drive_base:=true: all five controllers active,
no mesh or plugin errors, four wheels rendering with their tread, and a
lateral command turning all four to +90.0 deg both on screen and in the
joint states.

File: src/ranger_xarm_description/urdf/ranger_wheels.xacro (robot description, xacro)
@@ -2,26 +2,45 @@
 <robot xmlns:xacro="http://www.ros.org/wiki/xacro">
   <!-- Ranger Mini V3 four-wheel independent steering (4WIS) drive.
-       Geometry is measured off ranger_mini_v3_cad.stl rather than taken from
-       a datasheet, by least-squares circle fit to the lower arc of each tyre
-       (the arc nothing else can occlude). Fit residual is under 2 mm:
-         wheel radius   0.1026 m   (205 mm dia, the platform's 8" wheel)
-         wheelbase      0.494 m    (front axle +0.2461, rear -0.2479)
-         track          0.3704 m   (+/-0.1852)
+       Geometry is measured off ranger_mini_v3_cad.stl rather than taken
+       from a datasheet. The tyre is isolated as its own connected
+       component (scripts/split_wheel_meshes.py) and its axis fitted from
+       the tread, which makes it a clean cylinder to measure:
+         wheel radius   0.100036 m  (200 mm dia, the platform's stock wheel)
+         wheelbase      0.494 m     (+/-0.2470)
+         track          0.3704 m    (+/-0.1852)
          axle height    ground_z_nom + radius, so the tread sits exactly on
                         the documented ground plane instead of near it
-       Front/rear and left/right differ by 1-2 mm in the mesh, which is
-       tessellation noise on a symmetric platform, so the values above are
-       symmetrised; asymmetric wheelbase would otherwise show up as a
-       phantom yaw bias in the drive kinematics.
+       The radius previously read 0.1026 here, from a circle fit to "the
+       lower arc of each tyre" that had picked up the suspension sitting
+       inside the same envelope. The tread's own radius is 100.036 mm with
+       a 99.9th percentile of 100.032, and the lowest point of the whole
+       CAD is -327.029 mm, exactly ground_z. Those two give an axle at
+       -226.993 mm, which is where fitting the rear tyre's axis
+       independently puts it (-226.998). A 2.6 mm error is invisible on
+       screen but it scales every wheel speed the kinematics computes, so
+       on hardware the platform would have run 2.6% fast.
+       Front/rear and left/right differ by a few tenths of a millimetre in
+       the mesh, which is tessellation noise on a symmetric platform, so
+       the values above are symmetrised; an asymmetric wheelbase would
+       otherwise show up as a phantom yaw bias in the drive kinematics.
        Each corner is steer (revolute about Z, through the wheel centre) then
        roll (continuous about Y). Zero scrub radius: the real platform has a
        small caster offset, but modelling it buys nothing here and makes the
        inverse kinematics implicit rather than closed-form.
-       The wheels are COLLISION ONLY on purpose. ranger_mini_v3_cad.stl
-       already draws four wheels moulded into the chassis at zero steer; a
-       second set of visuals would render eight. The trade is that the wheels
-       do not visibly turn; verify steering from joint states, not the GUI. -->
+       The wheels used to be COLLISION ONLY, because ranger_mini_v3_cad.stl
+       draws four wheels moulded into the chassis and a second set of
+       visuals would have rendered eight. That made the robot look
+       completely static: the wheels you could see were welded to
+       base_link, and the ones that turned were invisible.
+       So the CAD is split instead. scripts/split_wheel_meshes.py cuts the
+       four wheels out as their own meshes and leaves a body mesh behind,
+       and each wheel is given to the link it belongs to. There are still
+       only four. Because wheel_link is a child of steer_link, one visual
+       shows both the roll and the steer.
+       A cylinder primitive would not have worked. A featureless cylinder
+       rotating about its own axis is indistinguishable from a stationary
+       one; it is the spokes and tread that make the rotation legible. -->
   <xacro:macro name="ranger_wheels" params="parent:='base_link' ground_z:=-0.327028595">
-    <xacro:property name="wheel_radius" value="0.1026"/>
+    <xacro:property name="wheel_radius" value="0.100036"/>
     <xacro:property name="wheel_width" value="0.070"/>
     <xacro:property name="half_wheelbase" value="0.2470"/>
@@ -82,4 +101,15 @@
              is that it cannot tip onto a tyre edge or climb a square lip,
              neither of which an empty ground plane offers. -->
+        <!-- The wheel cut out of the platform CAD, re-origined on its own
+             fitted axis of rotation so it spins true rather than wobbling.
+             Regenerate with scripts/split_wheel_meshes.py. -->
+        <visual name="${name}_wheel_visual">
+          <origin xyz="0 0 0" rpy="0 0 0"/>
+          <geometry>
+            <mesh filename="package://ranger_xarm_description/meshes/visual/ranger_wheel_${name}.stl"
+                  scale="0.001 0.001 0.001"/>
+          </geometry>
+          <material name="ranger_wheel_material"><color rgba="0.25 0.25 0.27 1"/></material>
+        </visual>
         <collision name="${name}_tyre">
           <origin xyz="0 0 0" rpy="0 0 0"/>

File: src/ranger_xarm_description/urdf/static_geometry.xacro (robot description, xacro)
@@ -17,10 +17,28 @@
         <inertia ixx="1.6086" ixy="0" ixz="0" iyy="3.1592" iyz="0" izz="3.5065"/>
       </inertial>
-      <visual name="ranger_cad_visual">
-        <geometry>
-          <mesh filename="package://ranger_xarm_description/meshes/visual/ranger_mini_v3_cad.stl" scale="0.001 0.001 0.001"/>
-        </geometry>
-        <material name="ranger_cad_material"><color rgba="0.72 0.72 0.68 1"/></material>
-      </visual>
+      <!-- Which CAD to draw depends on whether the wheels are their own
+           links. ranger_mini_v3_cad.stl is the whole vehicle with its
+           wheels moulded in at zero steer, which is right when nothing
+           else draws them. Once ranger_wheels.xacro provides real wheel
+           links, those moulded wheels are welded to base_link and sit on
+           top of the ones that actually turn, so the robot drives while
+           appearing completely static. The body mesh is the same CAD with
+           the four wheels cut out; see scripts/split_wheel_meshes.py. -->
+      <xacro:if value="${wheels_modelled}">
+        <visual name="ranger_cad_visual">
+          <geometry>
+            <mesh filename="package://ranger_xarm_description/meshes/visual/ranger_mini_v3_cad_body.stl" scale="0.001 0.001 0.001"/>
+          </geometry>
+          <material name="ranger_cad_material"><color rgba="0.72 0.72 0.68 1"/></material>
+        </visual>
+      </xacro:if>
+      <xacro:unless value="${wheels_modelled}">
+        <visual name="ranger_cad_visual">
+          <geometry>
+            <mesh filename="package://ranger_xarm_description/meshes/visual/ranger_mini_v3_cad.stl" scale="0.001 0.001 0.001"/>
+          </geometry>
+          <material name="ranger_cad_material"><color rgba="0.72 0.72 0.68 1"/></material>
+        </visual>
+      </xacro:unless>
       <xacro:if value="${use_collision}">
         <!-- ranger_envelope is the whole-vehicle bounding box, wheels

Commit message: Steer the knuckles, and hand gz its own resource path
Three things, all found by watching the sim rather than reading it.

**The knuckles did not steer.** Splitting the wheels out left the casting
above each one welded to base_link, so the wheel turned under a knuckle
that did not and the corner sheared visibly at full lock. The knuckles
are now cut from the CAD the same way and given to the steer links.

Which parts belong to a knuckle is less obvious than which belong to a
wheel, because a corner is thirty-odd components (flange, bolt circle,
motor housing, upright) rather than one, so they are selected by distance
from the steering axis. The threshold is not arbitrary. Between 20 and 40
mm the per-corner triangle count sits on a plateau at ~13050, varying
0.2% between corners, which is tessellation noise on a symmetric
platform. Widening to 60 mm jumps the count and makes the four corners
genuinely different (14547 vs 15739), which is chassis being dragged in.
30 mm sits mid-plateau. Visual only: the knuckle is clear of the ground,
and a collision there would only add contact pairs against the chassis it
is bolted to.

**gz could not find the arm's meshes.** sdformat rewrites package:// to
model:// when it converts the URDF, so gz resolves meshes by searching
GZ_SIM_RESOURCE_PATH for a directory named after the package. A package
only lands there if it exports a model path, and the vendored
xarm_description does not; upstream has no reason to, since it targets
the real arm. The result was 112 "Unable to find file with URI
[model://xarm_description/...]" errors and an arm with no visual meshes
at all, while the ranger meshes loaded fine because
ranger_xarm_description does carry the export. An invisible arm on a
visible robot is a poor first run for anyone cloning this.

sim.launch.py now hands gz every share directory on AMENT_PREFIX_PATH,
rather than patching someone else's package.xml. An existing value is
appended, so an overlay still wins. Verified by launching with
GZ_SIM_RESOURCE_PATH explicitly unset: 0 URI errors, all five controllers
active.

**The wheel radius is the unloaded one.** Recorded in the xacro and in
docs/TODO.md rather than guessed at. CAD does not sag; the real tyre
carries a quarter of ~100 kg and deflects, and both simulators inherit
the same optimism because the tyre is a rigid collision sphere in each.
The sign matters: omega = v / r, so a radius larger than the true rolling
radius makes the platform run slow and odometry over-report, which is
opposite to the 0.1026 error corrected in the previous commit, so the two
partly cancelled. Measuring it wants no instrumentation, just distance
divided by total wheel radians, which is deliberately clock-free.

Verified in gz with drive_base:=true, one instance, five controllers
active, zero mesh errors: a commanded spin turns all four wheels to
+/-53.1 deg and the knuckles turn with them.

File: src/ranger_xarm_description/urdf/ranger_wheels.xacro (robot description, xacro)
@@ -24,4 +24,24 @@
        the values above are symmetrised; an asymmetric wheelbase would
        otherwise show up as a phantom yaw bias in the drive kinematics.
+       Note this is the UNLOADED radius. It is a CAD dimension, and CAD
+       does not sag: on the real platform the tyre carries roughly a
+       quarter of ~100 kg and deflects, so its loaded rolling radius is
+       smaller than 100.036 mm by an amount nobody here has measured.
+       Both simulators inherit the same optimism, because the tyre is a
+       rigid collision sphere in each, so neither will ever show it.
+       The sign matters if this ever drives hardware. The kinematics turn
+       a commanded speed into a wheel rate as omega = v / r, so a radius
+       larger than the real rolling radius makes the platform run SLOW by
+       that ratio, and an odometry estimate built the same way reports
+       more distance than the platform travelled. That is the opposite
+       direction to the 0.1026 error corrected above, so the two partly
+       cancelled, which is a reason to measure rather than to leave both
+       in.
+       Measuring it wants no instrumentation: drive a straight line over
+       a known distance and count wheel revolutions, then r_eff is
+       distance / total radians. Deliberately a ratio of two measured
+       quantities with no clock in it, which is what makes it immune to
+       the sim-time trap documented in ranger_xarm_isaac's README, and it
+       is the same quantity that confirmed 0.1026 was wrong.
        Each corner is steer (revolute about Z, through the wheel centre) then
        roll (continuous about Y). Zero scrub radius: the real platform has a
@@ -61,4 +81,17 @@
           <inertia ixx="0.0015" ixy="0" ixz="0" iyy="0.0015" iyz="0" izz="0.0020"/>
         </inertial>
+        <!-- The steering casting, cut from the CAD like the wheel below it.
+             Without this the wheel turned under a knuckle that did not, and
+             the corner visibly sheared at full lock. No collision: the
+             knuckle is well clear of the ground, and a collision here would
+             only add contact pairs against the chassis it is bolted to. -->
+        <visual name="${name}_knuckle_visual">
+          <origin xyz="0 0 0" rpy="0 0 0"/>
+          <geometry>
+            <mesh filename="package://ranger_xarm_description/meshes/visual/ranger_knuckle_${name}.stl"
+                  scale="0.001 0.001 0.001"/>
+          </geometry>
+          <material name="ranger_knuckle_material"><color rgba="0.55 0.55 0.57 1"/></material>
+        </visual>
       </link>
       <joint name="${name}_steer_joint" type="revolute">

Commit message: Reconcile the 4WIS controllers and add a velocity wheel drive to gz
The isaac branch's ranger_4wis_controller.py had a command_mode (effort
or velocity) and its xacro a wheels_command_interface argument that the
public branch lacked. Both are ported, both default to effort, and the
default expanded URDF is byte-identical to before. Comments that said a
velocity command in gz is a rigid constraint now say what was actually
established: that is a bullet-featherstone behaviour, and the stale
'8 Nm' note on a 60 Nm joint limit is corrected.

sim.launch.py gains wheel_drive:=effort|velocity, which sets the xacro
interface, swaps the wheel controller to JointGroupVelocityController,
and puts the 4WIS controller in velocity mode. The default stays effort.

On dartsim the velocity drive does not reproduce the bullet failure: a
commanded spin in place yields 100 % of its yaw. On the rough-ground arc
it tracks every wheel to 0 % error with a fit residual of 0.001 m/s and
turns 134-135 deg of 137.5, against 83 deg for the stock effort loop and
without the chatter of a stiffened one. Rough-ground scores:

  wheel odometry  22.9-47.0 %  ->  3.5-8.4 %
  EKF             12.2-27.8 %  ->  0.77-1.84 %

comparable to Isaac (0.43-4.47 % / 0.54-2.89 %). The gz/Isaac gap was
the drive.

It is not the default yet because it regresses elsewhere. Flat-ground
wheel odometry picks up a constant +1.33 deg heading error, which a
per-segment breakdown puts almost entirely in the transition into the
crab (+2.03 deg): the stiff drive spins the wheels at full speed while
the knuckles are still sweeping to 90 deg. mixed_surface fails 3 of 5
trials (1 of 5 under effort) and low_friction EKF rises from 0.08 % to
0.44 %. The next step, recorded in docs/TODO.md, is to gate each wheel's
speed on its steering having converged.

run_surface_sweep.sh takes WHEEL_DRIVE from the environment, and
arc_probe.py accepts an arbitrary twist and labels its command column
honestly for either drive.

File: src/ranger_xarm_description/urdf/ranger_wheels.xacro (robot description, xacro)
@@ -162,14 +162,13 @@
         <origin xyz="0 0 0" rpy="0 0 0"/>
         <axis xyz="0 1 0"/>
-        <!-- 8 Nm is 78 N of thrust per wheel, ample for a 100 kg platform on
-             the flat, and the low value is deliberate. gz drives this joint
-             with a velocity motor, which is a near-rigid constraint on spin
-             rate; four of them plus four held steer angles over-determine a
-             3-DOF chassis, so any small steering error has the wheels
-             fighting each other instead of moving the robot. At 60 Nm the
-             motors always won and a commanded spin produced under 10% of
-             its yaw regardless of friction. Letting them be back-driven
-             lets the contact resolve the inconsistency, which is what a
-             real torque-driven wheel does. -->
+        <!-- The effort limit caps whatever drives this joint: the effort
+             command range, and on dartsim the force of a velocity servo.
+             History: under bullet-featherstone a velocity command was a
+             near-rigid motor constraint, and four of them plus four held
+             steer angles over-determined the 3-DOF chassis. With the limit
+             at 60 Nm a commanded spin produced under 10% of its yaw; an
+             8 Nm limit let the motors be back-driven and was tried as a
+             workaround before the wheels moved to effort control and the
+             engine to dartsim. -->
         <limit effort="60.0" velocity="25.0"/>
         <dynamics damping="0.02" friction="0.0"/>
@@ -214,5 +213,5 @@
        claims both silently runs the velocity law. Steering therefore claims
        position only and drive claims velocity only. -->
-  <xacro:macro name="ranger_wheels_ros2_control" params="name:='ranger_base' plugin">
+  <xacro:macro name="ranger_wheels_ros2_control" params="name:='ranger_base' plugin wheel_command:='effort'">
     <ros2_control name="${name}" type="system">
       <hardware>
@@ -244,8 +243,21 @@
              the speed loop. -->
         <joint name="${corner}_wheel_joint">
-          <command_interface name="effort">
-            <param name="min">-60.0</param>
-            <param name="max">60.0</param>
-          </command_interface>
+          <xacro:if value="${wheel_command == 'effort'}">
+            <command_interface name="effort">
+              <param name="min">-60.0</param>
+              <param name="max">60.0</param>
+            </command_interface>
+          </xacro:if>
+          <xacro:unless value="${wheel_command == 'effort'}">
+            <!-- A speed target for the simulator's joint velocity drive. In
+                 Isaac that is a PhysX drive; on dartsim it is a servo whose
+                 force is capped by the joint effort limit above, so the
+                 contact can still slip. The rigid-constraint failure
+                 described above is a bullet-featherstone behaviour. -->
+            <command_interface name="velocity">
+              <param name="min">-25.0</param>
+              <param name="max">25.0</param>
+            </command_interface>
+          </xacro:unless>
           <state_interface name="position"/>
           <state_interface name="velocity"/>

File: src/ranger_xarm_description/urdf/ranger_xarm.urdf.xacro (robot description, xacro)
@@ -57,4 +57,10 @@
   <xacro:arg name="fix_base_to_world" default="true"/>
   <xacro:arg name="wheels_ros2_control_plugin" default="gz_ros2_control/GazeboSimSystem"/>
+  <!-- How ros2_control commands the wheel joints. effort: torque, with the
+       speed loop closed in ranger_4wis_controller.py. velocity: wheel speed,
+       closed by the simulator's own torque-limited joint drive, as Isaac
+       does and as dartsim can. See ranger_wheels.xacro for why gz used
+       effort. -->
+  <xacro:arg name="wheels_command_interface" default="effort"/>
   <xacro:arg name="use_laptop_collision" default="true"/>
   <xacro:arg name="laptop_width" default="0.36"/><xacro:arg name="laptop_depth" default="0.25"/>
@@ -83,5 +89,6 @@
     <xacro:ranger_wheels parent="base_link" ground_z="${ground_z_nom}"/>
     <xacro:ranger_wheels_ros2_control name="ranger_base"
-      plugin="$(arg wheels_ros2_control_plugin)"/>
+      plugin="$(arg wheels_ros2_control_plugin)"
+      wheel_command="$(arg wheels_command_interface)"/>
   </xacro:if>
   <!-- Ground-projection reference, and the ROOT of the robot.
