Commit message: Give each wheel corner a sprung swing-arm suspension joint
The Ranger Mini 3.0 has independent swing-arm suspension, and a rigid
model does not behave like it on uneven ground: only two or three wheels
carry load at a time and a loaded wheel stalls while an unloaded one
spins. Each corner now rides on a vertical prismatic *_suspension_joint
between base_link and its steering knuckle: 15 mm of droop, 25 mm of
bump, a 20 kN/m spring preloaded to 12.5 mm of static sag and 570 N s/m
of damping. The static ride height is unchanged.

AgileX publishes no travel, rate or damping, so these are estimates to
replace with measurements on the robot. gz gets the spring through
springStiffness/springReference; for Isaac the USD converter reads the
same numbers. The joints are passive and declared to ros2_control with
state interfaces only, so robot_state_publisher gets them and nothing
commands them. use_suspension:=false restores the rigid corners.

File: src/ranger_xarm_description/urdf/ranger_wheels.xacro (robot description, xacro)
@@ -61,5 +61,34 @@
        rotating about its own axis is indistinguishable from a stationary
        one; it is the spokes and tread that make the rotation legible. -->
-  <xacro:macro name="ranger_wheels" params="parent:='base_link' ground_z:=-0.327028595">
+  <!-- Suspension. The Ranger Mini 3.0 has independent swing-arm suspension
+       (user manual V1.0.0, 2024.06: "Independent suspension"; datasheets:
+       "swing arm suspension"), and a rigid model does not behave like it
+       on uneven ground: only two or three wheels carry load at a time, and
+       a loaded wheel stalls while an unloaded one spins. Each corner rides
+       on a vertical prismatic joint (the swing arm's arc is short enough to
+       treat as a line at this travel), sprung and damped.
+       The manufacturer publishes no travel, rate or damping; these are
+       estimates to replace with measurements on the robot:
+         travel     15 mm of droop, 25 mm of bump about the static ride
+                    height (ground clearance is 105 mm);
+         spring     20 kN/m, a preloaded coil with 12.5 mm of static sag
+                    at ~25 kg per corner (4.5 Hz); its free length lies
+                    beyond full droop, so it pushes throughout the travel
+                    and never pulls a wheel up;
+         damping    570 N s/m, a damping ratio of ~0.4.
+       Stiff on purpose: at 8.2 kN/m the load moving onto the downhill
+       wheels across a side slope rolled the body several more degrees,
+       more when the springs reached their stops, enough to tip the robot
+       while crabbing.
+       The static ride height is unchanged: the joint's zero is where the
+       axle was, and the spring's reference (springReference, gz; the drive
+       target, Isaac) is 12.5 mm into droop. Positive is compression (the
+       wheel up into the chassis). -->
+  <xacro:macro name="ranger_wheels" params="parent:='base_link' ground_z:=-0.327028595 suspension:=true">
+    <xacro:property name="susp_droop" value="0.015"/>
+    <xacro:property name="susp_bump" value="0.025"/>
+    <xacro:property name="susp_sag" value="0.0125"/>
+    <xacro:property name="susp_stiffness" value="20000.0"/>
+    <xacro:property name="susp_damping" value="570.0"/>
     <xacro:property name="wheel_radius" value="0.100036"/>
     <xacro:property name="wheel_width" value="0.070"/>
@@ -95,8 +124,36 @@
         </visual>
       </link>
+      <xacro:if value="${suspension}">
+        <link name="${name}_suspension_link">
+          <inertial>
+            <origin xyz="0 0 0"/>
+            <mass value="0.3"/>
+            <inertia ixx="0.0002" ixy="0" ixz="0" iyy="0.0002" iyz="0" izz="0.0002"/>
+          </inertial>
+        </link>
+        <joint name="${name}_suspension_joint" type="prismatic">
+          <parent link="${parent}"/>
+          <child link="${name}_suspension_link"/>
+          <origin xyz="${x} ${y} ${axle_z}" rpy="0 0 0"/>
+          <axis xyz="0 0 1"/>
+          <limit lower="${-susp_droop}" upper="${susp_bump}" effort="5000.0" velocity="2.0"/>
+          <dynamics damping="${susp_damping}" friction="0.0"/>
+        </joint>
+        <gazebo reference="${name}_suspension_joint">
+          <springReference>${-susp_sag}</springReference>
+          <springStiffness>${susp_stiffness}</springStiffness>
+        </gazebo>
+      </xacro:if>
       <joint name="${name}_steer_joint" type="revolute">
-        <parent link="${parent}"/>
-        <child link="${name}_steer_link"/>
-        <origin xyz="${x} ${y} ${axle_z}" rpy="0 0 0"/>
+        <xacro:if value="${suspension}">
+          <parent link="${name}_suspension_link"/>
+          <child link="${name}_steer_link"/>
+          <origin xyz="0 0 0" rpy="0 0 0"/>
+        </xacro:if>
+        <xacro:unless value="${suspension}">
+          <parent link="${parent}"/>
+          <child link="${name}_steer_link"/>
+          <origin xyz="${x} ${y} ${axle_z}" rpy="0 0 0"/>
+        </xacro:unless>
         <axis xyz="0 0 1"/>
         <!-- 200 Nm is not the actuator's rating, it is what it takes to
@@ -213,5 +270,5 @@
        claims both silently runs the velocity law. Steering therefore claims
        position only and drive claims velocity only. -->
-  <xacro:macro name="ranger_wheels_ros2_control" params="name:='ranger_base' plugin wheel_command:='effort'">
+  <xacro:macro name="ranger_wheels_ros2_control" params="name:='ranger_base' plugin wheel_command:='effort' suspension:=true">
     <ros2_control name="${name}" type="system">
       <hardware>
@@ -263,4 +320,12 @@
           <state_interface name="velocity"/>
         </joint>
+        <!-- Passive: states only, so robot_state_publisher gets the joint
+             (every link below it hangs off it) and nothing commands it. -->
+        <xacro:if value="${suspension}">
+          <joint name="${corner}_suspension_joint">
+            <state_interface name="position"/>
+            <state_interface name="velocity"/>
+          </joint>
+        </xacro:if>
       </xacro:macro>
       <xacro:corner_ifaces corner="front_left"/>

File: src/ranger_xarm_description/urdf/ranger_xarm.urdf.xacro (robot description, xacro)
@@ -55,4 +55,7 @@
   <xacro:arg name="gz_sensors" default="false"/>
   <xacro:arg name="use_wheels" default="false"/>
+  <!-- A sprung vertical joint per corner (the swing-arm suspension); see
+       ranger_wheels.xacro. -->
+  <xacro:arg name="use_suspension" default="true"/>
   <xacro:arg name="fix_base_to_world" default="true"/>
   <xacro:arg name="wheels_ros2_control_plugin" default="gz_ros2_control/GazeboSimSystem"/>
@@ -87,8 +90,10 @@
   </xacro:if>
   <xacro:if value="$(arg use_wheels)">
-    <xacro:ranger_wheels parent="base_link" ground_z="${ground_z_nom}"/>
+    <xacro:ranger_wheels parent="base_link" ground_z="${ground_z_nom}"
+      suspension="$(arg use_suspension)"/>
     <xacro:ranger_wheels_ros2_control name="ranger_base"
       plugin="$(arg wheels_ros2_control_plugin)"
-      wheel_command="$(arg wheels_command_interface)"/>
+      wheel_command="$(arg wheels_command_interface)"
+      suspension="$(arg use_suspension)"/>
   </xacro:if>
   <!-- Ground-projection reference, and the ROOT of the robot.
